File: Tilt Table, V3/Summer Board.sch (EAGLE design)
At the start: 8 parts, among them X1 0446200002, X3 SPB5

Commit message: ATmega328 reference design
Parts:
- removed X3: SPB5, con-hirschmann:SPB5
- added JS: PINS_5SILK, nolan-utsa:PINS_5SILK
- renumbered U$1 to Y-SERVO, U$2 to X-SERVO
Connections:
- net 3.3V: now also JS.2; no longer X3.2
- net GND: now also JS.1; no longer X3.1
- net X_ANA: now also JS.3; no longer X3.3
- net Y_ANA: now also JS.4; no longer X3.4
Changed lines of the file:
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@@
 <parts>
 <part name="FRDM1" library="nolan-utsa" deviceset="FRDM-KL25Z" device="NORMAL"/>
-<part name="U$1" library="nolan-utsa" deviceset="PINS_3" device="_2.54"/>
-<part name="U$2" library="nolan-utsa" deviceset="PINS_3" device="_2.54"/>
+<part name="Y-SERVO" library="nolan-utsa" deviceset="PINS_3" device="_2.54"/>
+<part name="X-SERVO" library="nolan-utsa" deviceset="PINS_3" device="_2.54"/>
 <part name="U$3" library="nolan-utsa" deviceset="PINS_4" device="SILK"/>
 <part name="X1" library="con-molex" library_urn="urn:adsk.eagle:library:165" deviceset="0446200002" device="" package3d_urn="urn:adsk.eagle:package:8078921/1"/>
@@
 <part name="GND6" library="nolan-utsa" deviceset="GND" device=""/>
 <part name="X2" library="con-wago-500" library_urn="urn:adsk.eagle:library:195" deviceset="W237-102" device="" package3d_urn="urn:adsk.eagle:package:10688/1"/>
-<part name="X3" library="con-hirschmann" library_urn="urn:adsk.eagle:library:153" deviceset="SPB5" device="" package3d_urn="urn:adsk.eagle:package:7457/1"/>
 <part name="GND7" library="supply1" library_urn="urn:adsk.eagle:library:371" deviceset="GND" device=""/>
+<part name="JS" library="nolan-utsa" deviceset="PINS_5" device="SILK"/>
 </parts>
 <sheets>
@@
 <attribute name="NAME" x="111.76" y="157.48" size="2.032" layer="95"/>
 </instance>
-<instance part="U$1" gate="G$1" x="165.1" y="27.94" smashed="yes" rot="R180">
+<instance part="Y-SERVO" gate="G$1" x="165.1" y="27.94" smashed="yes" rot="R180">
 <attribute name="NAME" x="167.64" y="17.78" size="1.778" layer="95" ratio="13" rot="R180"/>
 <attribute name="VALUE" x="167.64" y="20.32" size="1.778" layer="96" ratio="13" rot="R180"/>
 </instance>
-<instance part="U$2" gate="G$1" x="165.1" y="50.8" smashed="yes" rot="R180">
+<instance part="X-SERVO" gate="G$1" x="165.1" y="50.8" smashed="yes" rot="R180">
 <attribute name="NAME" x="167.64" y="40.64" size="1.778" layer="95" ratio="13" rot="R180"/>
 <attribute name="VALUE" x="167.64" y="43.18" size="1.778" layer="96" ratio="13" rot="R180"/>
@@
 <attribute name="NAME" x="30.48" y="38.989" size="1.778" layer="95" rot="R180"/>
 </instance>
-<instance part="X3" gate="1" x="58.42" y="147.32" smashed="yes">
-<attribute name="VALUE" x="55.88" y="137.16" size="1.778" layer="96"/>
-<attribute name="NAME" x="55.88" y="155.575" size="1.778" layer="95"/>
-</instance>
-<instance part="GND7" gate="1" x="68.58" y="152.4" smashed="yes" rot="R90">
-<attribute name="VALUE" x="71.12" y="149.86" size="1.778" layer="96" rot="R90"/>
+<instance part="GND7" gate="1" x="55.88" y="152.4" smashed="yes" rot="R90">
+<attribute name="VALUE" x="58.42" y="149.86" size="1.778" layer="96" rot="R90"/>
+</instance>
+<instance part="JS" gate="G$1" x="43.18" y="147.32" smashed="yes">
+<attribute name="NAME" x="40.64" y="160.02" size="1.778" layer="95" ratio="13"/>
+<attribute name="VALUE" x="40.64" y="157.48" size="1.778" layer="96" ratio="13"/>
 </instance>
 </instances>
@@
 </segment>
 <segment>
-<pinref part="U$2" gate="G$1" pin="1"/>
+<pinref part="X-SERVO" gate="G$1" pin="1"/>
 <pinref part="GND9" gate="1" pin="GND"/>
 </segment>
 <segment>
-<pinref part="U$1" gate="G$1" pin="1"/>
+<pinref part="Y-SERVO" gate="G$1" pin="1"/>
 <pinref part="GND10" gate="1" pin="GND"/>
 </segment>
@@
 </segment>
 <segment>
-<pinref part="X3" gate="1" pin="1"/>
 <pinref part="GND7" gate="1" pin="GND"/>
-<wire x1="63.5" y1="152.4" x2="66.04" y2="152.4" width="0.1524" layer="91"/>
+<pinref part="JS" gate="G$1" pin="1"/>
+<wire x1="50.8" y1="152.4" x2="53.34" y2="152.4" width="0.1524" layer="91"/>
 </segment>
 </net>
@@
 <net name="PTB0" class="0">
 <segment>
-<pinref part="U$2" gate="G$1" pin="3"/>
+<pinref part="X-SERVO" gate="G$1" pin="3"/>
 <wire x1="157.48" y1="53.34" x2="154.94" y2="53.34" width="0.1524" layer="91"/>
 <wire x1="154.94" y1="53.34" x2="154.94" y2="55.88" width="0.1524" layer="91"/>
@@
 <net name="PTB1" class="0">
 <segment>
-<pinref part="U$1" gate="G$1" pin="3"/>
+<pinref part="Y-SERVO" gate="G$1" pin="3"/>
 <wire x1="157.48" y1="30.48" x2="154.94" y2="30.48" width="0.1524" layer="91"/>
 <wire x1="154.94" y1="30.48" x2="154.94" y2="33.02" width="0.1524" layer="91"/>
@@
 <net name="N$2" class="0">
 <segment>
-<pinref part="U$2" gate="G$1" pin="2"/>
+<pinref part="X-SERVO" gate="G$1" pin="2"/>
 <wire x1="139.7" y1="50.8" x2="157.48" y2="50.8" width="0.1524" layer="91"/>
 <wire x1="139.7" y1="50.8" x2="139.7" y2="27.94" width="0.1524" layer="91"/>
 <wire x1="139.7" y1="27.94" x2="157.48" y2="27.94" width="0.1524" layer="91"/>
-<pinref part="U$1" gate="G$1" pin="2"/>
+<pinref part="Y-SERVO" gate="G$1" pin="2"/>
 <pinref part="U$4" gate="G$1" pin="OUT+"/>
 <wire x1="129.54" y1="50.8" x2="139.7" y2="50.8" width="0.1524" layer="91"/>
@@
 <net name="3.3V" class="0">
 <segment>
-<pinref part="X3" gate="1" pin="2"/>
-<wire x1="63.5" y1="149.86" x2="78.74" y2="149.86" width="0.1524" layer="91"/>
-<wire x1="78.74" y1="149.86" x2="78.74" y2="152.4" width="0.1524" layer="91"/>
-<label x="78.74" y="152.4" size="1.778" layer="95" xref="yes"/>
+<wire x1="50.8" y1="149.86" x2="86.36" y2="149.86" width="0.1524" layer="91"/>
+<label x="86.36" y="149.86" size="1.778" layer="95" xref="yes"/>
+<pinref part="JS" gate="G$1" pin="2"/>
 </segment>
 <segment>
@@
 <net name="X_ANA" class="0">
 <segment>
-<pinref part="X3" gate="1" pin="3"/>
-<wire x1="63.5" y1="147.32" x2="78.74" y2="147.32" width="0.1524" layer="91"/>
-<wire x1="78.74" y1="147.32" x2="78.74" y2="144.78" width="0.1524" layer="91"/>
-<label x="78.74" y="144.78" size="1.778" layer="95" xref="yes"/>
+<wire x1="50.8" y1="147.32" x2="71.12" y2="147.32" width="0.1524" layer="91"/>
+<label x="71.12" y="147.32" size="1.778" layer="95" xref="yes"/>
+<pinref part="JS" gate="G$1" pin="3"/>
 </segment>
 <segment>
@@
 <net name="Y_ANA" class="0">
 <segment>
-<pinref part="X3" gate="1" pin="4"/>
-<wire x1="63.5" y1="144.78" x2="73.66" y2="144.78" width="0.1524" layer="91"/>
-<wire x1="73.66" y1="144.78" x2="73.66" y2="142.24" width="0.1524" layer="91"/>
-<label x="73.66" y="142.24" size="1.778" layer="95" rot="R180" xref="yes"/>
-</segment>
-<segment>
+<label x="58.42" y="144.78" size="1.778" layer="95" xref="yes"/>
+<pinref part="JS" gate="G$1" pin="4"/>
+<wire x1="50.8" y1="144.78" x2="58.42" y2="144.78" width="0.1524" layer="91"/>
+</segment>
+<segment>
