File: VIVA_PIC16/V5/VIVA_PIC16_V5.sch (EAGLE design)
At the start: 42 parts, among them J101 2.1MMJACKTHM, J102 1X2-3.5MM-3.5MM, J103 PINS_2, J104 PINS_32.54, J201 VIVA_PIC16, J202 VIVA-HEADER-ADCNONAME, J203 PICKIT3, J204 PINS_32.54, M101 VIVA_USB-TTL, Q101 2N3906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

Commit message: *
Other:
- note added: "ARDUINO SECTION"
- note added: "VIVA Header"
- note removed: "1.0"
- note removed: "4.2"
- note removed: "Author"
- note removed: "Document"
- note removed: "Microcontroller"
- note removed: "Nolan Manteufel"
- note removed: "Page"
- note removed: "Power, USB Module, High-side Switch"
- note removed: "REV."
- note removed: "Revision Date"
- note removed: "SHEET"
- note removed: "UTSA PORTION"
- note removed: "VIVA Headers"
- note removed: "VIVA PORTION"
- moved on the sheet: LED201, R201, R202, R203
