File: VIVA_PIC16/Rev 5.0/v5.sch (EAGLE design)
At the start: 55 parts, among them J102 1X2-3.5MM-3.5MM, J103 PINS_2, J201 VIVA_PIC16, J202 VIVA-HEADER-ADCNONAME, J203 PICKIT3, J204 PINS_32.54, M101 VIVA_USB-TTL, Q101 2N3906, Q102 2N3904, SW1. OS202013MT5QN1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

Commit message: ATmega PN
Other:
- note added: "ATMEGA328PB-AU"
Changed lines of the file:
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@@
 <sheet>
 <plain>
+<text x="48.26" y="132.08" size="1.778" layer="91">ATMEGA328PB-AU</text>
 </plain>
 <instances>
