File: VIVA_PIC16/Rev 5.0/v5.sch (EAGLE design)
At the start: 24 parts, among them SW1. OS202013MT5QN1, U2 AMS1117-3.3, U3 TP4056, U5 AP1603

Commit message: v5 draft
Parts:
- removed D3, D4: 1N5819, utsa:DIODE-SOD80C
- removed U5: AP1603, utsa:AP1603
- added B201: (no value), nolan-utsa:PUSHBUTTON6X6MM
- added C10: 1u, utsa:C0805
- added C2: 10u, 1206, utsa:C-EUC1206
- added C201, C202: 4u7, nolan-utsa:C0805
- added C203: 1u, nolan-utsa:C0805
- added D1, D2: 1N5819, utsa:DIODE-SOD80C
- added J102: 1X2-3.5MM-3.5MM, nolan-utsa:1X2-3.5MM-3.5MM
- added J103: PINS_2, nolan-utsa:PINS_2
- added J201: VIVA_PIC16, nolan-viva:VIVA_PIC16
- added J202: VIVA-HEADER-ADCNONAME, nolan-utsa:VIVA-HEADER-ADCNONAME
- added J203: PICKIT3, nolan-viva:PICKIT3
- added J204: PINS_32.54, nolan-utsa:PINS_32.54
- added LED201: Hello World!, nolan-utsa:RGB_LED
- added M101: VIVA_USB-TTL, nolan-utsa:VIVA_USB-TTL
- added PIC: PIC16F1829, nolan-utsa:PIC16F1829
- added Q101: 2N3906, nolan-utsa:2N3906SOT23
- added Q102: 2N3904, nolan-utsa:2N3904SOT23
- added R101, R207: 10k, adafruit:R-US_R0805
- added R102, R206: 100k, adafruit:R-US_R0805
- added R103: 1k, adafruit:R-US_R0805
- added R104: 4k7, adafruit:R-US_R0805
- added R201, R202, R203: 150, adafruit:R-US_R0805
- added R204, R205: 2k2, adafruit:R-US_R0805
- added TP1, TP2: (no value), nolan-utsa:TESTPOINTFIDUCIAL
- added U$201: VIVA_UTSA-KEYPAD, nolan-utsa:VIVA_UTSA-KEYPAD
- added U1: TP4056, utsa:TP4056
- C1: value 47u -> 10u, 1206; device utsa:C-EU865080642006 -> utsa:C-EUC1206
- C4: value 1u -> 47u; device utsa:C0805 -> utsa:C-EU865080642006
- C5: value 10u, 1206 -> 1u; device utsa:C-EUC1206 -> utsa:C0805
- C6: value 10u, 1206 -> 47u; device utsa:C-EUC1206 -> utsa:C-EU865080642006
- C9: value 47u -> 1u; device utsa:C-EU865080642006 -> utsa:C0805
- R1: value 1k -> RPROG
- R3: value RPROG -> 1k
- U2: value AMS1117-3.3 -> AP1603; device utsa:REGULATOR_SCHLM1117 -> utsa:AP1603
- U3: value TP4056 -> AMS1117-3.3; device utsa:TP4056 -> utsa:REGULATOR_SCHLM1117
Connections:
- removed net DCDC_5V: C9.1, L2.2, U5.5.OUT
- new net B+_FUSED: C4.1, C5.+, F1.2, L1.1
- new net DCDC_OUT: C6.1, C7.+, L2.2, U2.5.OUT
- new net DCDC_REF: C3.+, U2.3.REF
- new net ICSP_CLK: J201.18, J203.5.PGC, PIC.18.RA1/ICSPCLK
- new net ICSP_DAT: J201.19, J203.4.PGD, PIC.19.RA0/ICSPDAT
- new net MCLR: J201.4, J203.1.MCLR, J204.3, PIC.4.RA3/MCLR, R207.2
- new net N$10: Q102.B, R103.2
- new net N$11: LED201.4.B-, R201.1
- new net N$12: LED201.2.G-, R202.1
- new net N$13: LED201.1.R-, R203.1
- new net N$14: M101.(1)3V3
- new net N$15: J102.2, Q101.C
- new net N$16: M101.(6)5V
- new net N$6: J103.1, J103.2, R103.1, R104.2
- new net N$9: Q101.E, R102.1
- new net RA2: J201.17, PIC.17.RA2, R201.2
- new net RA4: J201.3, PIC.3.RA4, U$201.1
- new net RA5: J201.2, PIC.2.RA5, R202.2
- new net RB4: J201.13, PIC.13.RB4, R204.2
- new net RB5: J201.12, J202.5.ADC2, PIC.12.RB5
- new net RB6: J201.11, PIC.11.RB6, R205.2
- new net RB7: J201.10, J204.1, PIC.10.RB7
- new net RC0: J201.16, PIC.16.RC0, U$201.4
- new net RC1: J201.15, PIC.15.RC1, U$201.3
- new net RC2: J201.14, J202.3.ADC0, PIC.14.RC2
- new net RC3: J201.7, J202.4.ADC1, PIC.7.RC3
- new net RC4: J201.6, M101.(3)RX.I, PIC.6.RC4
- new net RC5: J201.5, M101.(4)TX.O, PIC.5.RC5
- new net RC6: J201.8, PIC.8.RC6, R203.2
- new net RC7: J201.9, PIC.9.RC7, U$201.2
- new net SWITCH_NODE: L1.2, U2.4.LX
- new net VDD: C201.P$2, C202.P$2, C203.P$2, J201.1, J202.2.VDD, J203.2.VDD(PWR), LED201.3.+, PIC.1.VDD, R204.1, R205.1, R206.1, R207.1
- net +3V3: now also C10.+, U3.OUT; no longer C4.+, U2.OUT
- net +5V: now also C8.1, C9.+, U3.IN; no longer C1.1, C3.+, U2.IN
- net B+: now also C2.1, U1.5.BAT; no longer C6.1, U3.5.BAT
- net CHARGE: now also R3.2, U1.7.CHRG; no longer R2.2, U3.7.CHRG
- net DCDC_ENABLE: now also U2.6.EN; no longer U5.6.EN
- net GND: now also B201.1, C10.-, C2.2, C201.P$1, C202.P$1, C203.P$1, C4.2, C5.-, C9.-, J102.1, J201.20, J202.1.GND, J203.3.VSS(GND), PIC.20.VSS, Q102.E, R1.1, R104.1, U1.1.TEMP, U1.3.GND, U2.1.FB, U2.2.GND, U3.GND; no longer C4.-, C5.2, C9.2, R3.1, U2.GND, U3.1.TEMP, U3.3.GND, U5.1.FB, U5.2.GND
- net N$1: now also B201.2, J204.2, R206.2; no longer L1.2, U5.4.LX
- net N$2: now also R2.1; no longer R1.1
- net N$3: now also R3.1; no longer R2.1
- net N$5: now also Q101.B, R101.2; no longer C8.1, F1.2, L1.1
- net N$7: now also R1.2, U1.2.PROG; no longer R3.2, U3.2.PROG
- net N$8: now also Q102.C, R101.1, R102.2; no longer C7.+, U5.3.REF
- net STANDBY: now also R2.2, U1.6.STDBY; no longer R1.2, U3.6.STDBY
- net USB_5V_AT: now also D1.A; no longer D3.A
- net USB_5V_PIC: now also D2.A; no longer D4.A
- net VCC: now also C1.1, D1.C, D2.C, U1.4.VCC, U1.8.ENABLE; no longer C5.1, D3.C, D4.C, U3.4.VCC, U3.8.ENABLE
Other:
- note added: "Capacitance Keypad"
- note added: "Fiducials"
- note added: "Hello World LED"
- note added: "NOTES: (1) Shielded end of switching power supply inductor is connected to switch node."
- note added: "PIC Microcontroller"
- note added: "PIC16 Headers"
- note added: "PICkit3 Header"
- note added: "Push Button"
- note added: "VIVA Headers"
- note removed: "NOTES: (1) Shielded end of switching power supply inductor is connected to switch node. (2) In PCB layout, size of switch node is minimized. (3) In PCB layout, component pads on switch node do not have thermal reliefs."

Commit message: *
Parts:
- removed C201, C202: 4u7, nolan-utsa:C0805
- removed C203: 1u, nolan-utsa:C0805
- removed J102: 1X2-3.5MM-3.5MM, nolan-utsa:1X2-3.5MM-3.5MM
- removed J103: PINS_2, nolan-utsa:PINS_2
- removed J201: VIVA_PIC16, nolan-viva:VIVA_PIC16
- removed J204: PINS_32.54, nolan-utsa:PINS_32.54
- removed M101: VIVA_USB-TTL, nolan-utsa:VIVA_USB-TTL
- removed PIC: PIC16F1829, nolan-utsa:PIC16F1829
- removed Q101: 2N3906, nolan-utsa:2N3906SOT23
- removed Q102: 2N3904, nolan-utsa:2N3904SOT23
- removed R101, R207: 10k, adafruit:R-US_R0805
- removed R102, R206: 100k, adafruit:R-US_R0805
- removed R103: 1k, adafruit:R-US_R0805
- removed R104: 4k7, adafruit:R-US_R0805
- removed R201, R202, R203: 150, adafruit:R-US_R0805
- removed R204, R205: 2k2, adafruit:R-US_R0805
- removed TP1, TP2: (no value), nolan-utsa:TESTPOINTFIDUCIAL
- removed U$201: VIVA_UTSA-KEYPAD, nolan-utsa:VIVA_UTSA-KEYPAD
- added C11, C12, C13, C14, C15: 1u, utsa:C0805
- added FIDUCIAL1, FIDUCIAL2: (no value), utsa:FIDUCIAL
- added J1: Transmitter, utsa:VIVA-HEADER-GPIO-1
- added J2: Receiver, utsa:VIVA-HEADER-RF-RX
- added J3: Pushbutton Jumper, utsa:PINS_3_2.54
- added R10, R9: 2k2, utsa:R-EU__R0805
- added R4, R5, R6: 150, utsa:R-EU__R0805
- added R7, R8: 10k, utsa:R-EU__R0805
- added U$11: VIVA_USB-TTL, utsa:VIVA_USB-TTL
- added U$6: VIVA_PIC16BOARD, utsa:VIVA_PIC16BOARD
- added U$7: VIVA_UTSA-KEYPADV5, utsa:VIVA_UTSA-KEYPADV5
- added U4: PIC16F1829, utsa:PIC16F1829300
Connections:
- removed net N$10: Q102.B, R103.2
- removed net N$11: LED201.4.B-, R201.1
- removed net N$12: LED201.2.G-, R202.1
- removed net N$13: LED201.1.R-, R203.1
- removed net N$15: J102.2, Q101.C
- removed net N$8: Q102.C, R101.1, R102.2
- removed net N$9: Q101.E, R102.1
- new net N$4: LED201.2.G-, R5.2
- net GND: now also C11.-, C12.-, C13.-, C14.-, C15.-, U$6.20, U4.20.VSS; no longer C201.P$1, C202.P$1, C203.P$1, J102.1, J201.20, PIC.20.VSS, Q102.E, R104.1
- net ICSP_CLK: now also U$6.18, U4.18.RA1/ICSPCLK; no longer J201.18, PIC.18.RA1/ICSPCLK
- net ICSP_DAT: now also U$6.19, U4.19.RA0/ICSPDAT; no longer J201.19, PIC.19.RA0/ICSPDAT
- net MCLR: now also J3.3, R7.2, U$6.4, U4.4.RA3/MCLR; no longer J201.4, J204.3, PIC.4.RA3/MCLR, R207.2
- net N$1: now also J3.2, R8.2; no longer J204.2, R206.2
- net N$14: now also U$11.(1)3V3; no longer M101.(1)3V3
- net N$16: now also U$11.(6)5V; no longer M101.(6)5V
- net N$5: now also LED201.1.R-, R6.2; no longer Q101.B, R101.2
- net N$6: now also LED201.4.B-, R4.2; no longer J103.1, J103.2, R103.1, R104.2
- net RA2: now also R4.1, U$6.17, U4.17.RA2; no longer J201.17, PIC.17.RA2, R201.2
- net RA4: now also U$6.3, U$7.1, U4.3.RA4; no longer J201.3, PIC.3.RA4, U$201.1
- net RA5: now also R5.1, U$6.2, U4.2.RA5; no longer J201.2, PIC.2.RA5, R202.2
- net RB4: now also R10.2, U$6.13, U4.13.RB4; no longer J201.13, PIC.13.RB4, R204.2
- net RB5: now also U$6.12, U4.12.RB5; no longer J201.12, PIC.12.RB5
- net RB6: now also R9.2, U$6.11, U4.11.RB6; no longer J201.11, PIC.11.RB6, R205.2
- net RB7: now also J3.1, U$6.10, U4.10.RB7; no longer J201.10, J204.1, PIC.10.RB7
- net RC0: now also U$6.16, U$7.4, U4.16.RC0; no longer J201.16, PIC.16.RC0, U$201.4
- net RC1: now also U$6.15, U$7.3, U4.15.RC1; no longer J201.15, PIC.15.RC1, U$201.3
- net RC2: now also U$6.14, U4.14.RC2; no longer J201.14, PIC.14.RC2
- net RC3: now also U$6.7, U4.7.RC3; no longer J201.7, PIC.7.RC3
- net RC4: now also U$11.(3)MCU.TX, U$6.6, U4.6.RC4; no longer J201.6, M101.(3)RX.I, PIC.6.RC4
- net RC5: now also U$11.(4)MCU.RX, U$6.5, U4.5.RC5; no longer J201.5, M101.(4)TX.O, PIC.5.RC5
- net RC6: now also R6.1, U$6.8, U4.8.RC6; no longer J201.8, PIC.8.RC6, R203.2
- net RC7: now also U$6.9, U$7.2, U4.9.RC7; no longer J201.9, PIC.9.RC7, U$201.2
- net VDD: now also C11.+, C12.+, C13.+, C14.+, C15.+, R10.1, R7.1, R8.1, R9.1, U$6.1, U4.1.VDD; no longer C201.P$2, C202.P$2, C203.P$2, J201.1, PIC.1.VDD, R204.1, R205.1, R206.1, R207.1
Other:
- note added: "Programming Header"
- note added: "VIVA Header: ANALOG"
- note added: "VIVA Header: RECEIVER e.g. MX-05V"
- note added: "VIVA Header: TRANSMITTER e.g. MX-FS-03V"
- note removed: "PICkit3 Header"
- note removed: "VIVA Headers"
