File: VIVA_PIC16/Rev 5.0/v5.sch (EAGLE design)
At the start: 31 parts, among them J1 VDD Selector, J2 Transmitter, J3 Receiver, J4 PICKIT3, J5 VIVA-HEADER-ADCNONAME, U1 VIVA_UTSA-KEYPADV5, U2 VIVA_USB-TTL, U3 PIC16F1829, U4 VIVA-HEADER-I2C-RA, U5 VIVA_PIC16BOARD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

Commit message: *
Parts:
- added C7, C8: (no value), utsa:C0805
- added J6: ICSP, utsa:PINS_6-2X3
- added J7, J8: PINS_162X8, utsa:PINS_162X8
- added U$2: VIVA-HEADER-UART-XS, utsa:VIVA-HEADER-UART-XS
- added U$3: VIVA_OLED, utsa:VIVA_OLED
- added XTAL1: (no value), utsa:CRYSTAL-SMD
- J5: value VIVA-HEADER-ADCNONAME -> (none); device nolan-utsa:VIVA-HEADER-ADCNONAME -> utsa:VIVA-HEADER-ADC-PIC16
- LED1: value Hello World! -> (none); device nolan-utsa:RGB_LED -> utsa:LED_RGBLTST-C19FD1WT
Connections:
- removed net N$5 (its old number): LED1.1.R-, R3.2
- new net AT_MISO: J6.1, U6.PB6
- new net AT_MOSI: J6.4, U6.PB5
- new net AT_RESET: J6.5
- new net AT_RST: U6.PC6
- new net AT_SCK: J6.3, U6.PB7
- new net AT_VTG: J6.2
- new net N$2: C7.+, XTAL1.2
- new net N$3: C8.+, XTAL1.1
- new net N$4: LED1.1.R-, R1.2
- net GND: now also C7.-, C8.-, J6.6
- net N$6: now also R3.2; no longer R1.2
- net RA2: now also R3.1; no longer R1.1
- net RC6: now also R1.1; no longer R3.1
Other:
- note removed: "ATMEGA328PB-AU"

Commit message: *
Parts:
- removed J2: Transmitter, utsa:VIVA-HEADER-GPIO-1
- removed J3: Receiver, utsa:VIVA-HEADER-RF-RX
- added B3: (no value), nolan-utsa:PUSHBUTTON6X6MM
- added C10: 10u, utsa:C-EU_C0805
- added C11: 100n, utsa:C-EU_C0805
- added C12, C13: (no value), utsa:C0805
- added C9: 1u, utsa:C0805
- added J10: ADC7, utsa:VIVA-HEADER-GPIO-1
- added J11: ADC6, utsa:VIVA-HEADER-GPIO-1
- added J9: (no value), utsa:VIVA-HEADER-ADC-PIC16
- added R10, R13, R9: 10k, utsa:R-EU__R0805
- added R11, R12: 10, utsa:R-EU__R0805
- added U7: VIVA_USB-TTL, utsa:VIVA_USB-TTL
Connections:
- net N$1 renamed MCLR_CAP
- removed net N$2: C7.+, XTAL1.2
- removed net N$3: C8.+, XTAL1.1
- removed net RB4: R5.2, U3.13.RB4, U4.3.SDA, U5.13
- removed net RB6: R6.2, U3.11.RB6, U4.4.SCL, U5.11
- new net ADC6: J11.3.DATA, U6.ADC6
- new net ADC7: J10.3.DATA, U6.ADC7
- new net AREF: C10.2, C11.2, R12.2, U6.AREF
- new net AT_RST_BTN: B3.2, R13.1, R9.2
- new net AT_RST_CAP: C9.+, R10.2, R9.1
- new net AT_RXD: U6.PD0, U7.(4)MCU.RX
- new net AT_TXD: U6.PD1, U7.(3)MCU.TX
- new net AVCC: C10.1, C11.1, R11.2, U6.AVCC
- new net PC0: J9.3.ADC0, U6.PC0
- new net PC1: J9.4.ADC1, U6.PC1
- new net PC2: J9.5.ADC2, U6.PC2
- new net SCL: R6.2, U$3.3.SCL, U3.11.RB6, U4.4.SCL, U5.11, U6.PC5
- new net SDA: R5.2, U$3.4.SDA, U3.13.RB4, U4.3.SDA, U5.13, U6.PC4
- new net XTAL1: C7.+, U6.PB6, XTAL1.2
- new net XTAL2: C8.+, U6.PB7, XTAL1.1
- net +3V3: now also U7.(1)3V3
- net +5V: now also U7.(6)5V
- net AT_MISO: now also U6.PB4; no longer U6.PB6
- net AT_MOSI: now also U6.PB3; no longer U6.PB5
- net AT_RST: now also R13.2
- net AT_SCK: now also U6.PB5; no longer U6.PB7
- net GND: now also B3.1, C12.-, C13.-, C9.-, J10.1.GND, J11.1.GND, J9.1.GND, R12.1, U$3.2.GND, U7.(5)GND; no longer J2.1.GND, J3.1.GND, U6.AREF
- net VDD: now also C12.+, C13.+, J10.2.VDD, J11.2.VDD, J9.2.VDD, R10.1, R11.1, U$3.1.VDD; no longer J2.2.VDD, J3.2.VDD, U6.AVCC
Other:
- note added: "433MHz RECEIVER: MX-05V"
- note added: "433MHz TRANSMITTER: MX-FS-03V"
- note removed: "VIVA Header: RECEIVER e.g. MX-05V"
- note removed: "VIVA Header: TRANSMITTER e.g. MX-FS-03V"
- moved on the sheet: C7, C8, J7, J8, XTAL1
