File: VIVA_PIC16/Rev 5.0/v5.brd (EAGLE design)
At the start: 100 x 100 mm, 24 parts, among them SW1. OS202013MT5QN1, U2 AMS1117-3.3, U3 TP4056, U5 AP1603

Commit message: v5 draft
Parts:
- removed D3, D4: 1N5819, utsa:SOD80C
- removed U5: AP1603, utsa:SOT23-6
- added B201: (no value), nolan-utsa:6X6MM
- added C10: 1u, utsa:C0805
- added C2: 10u, 1206, utsa:C1206
- added C201, C202: 4u7, nolan-utsa:C0805
- added C203: 1u, nolan-utsa:C0805
- added D1, D2: 1N5819, utsa:SOD80C
- added J102: 1X2-3.5MM-3.5MM, nolan-utsa:1X2-3.5MM
- added J103: PINS_2, nolan-utsa:PINS_2
- added J201: VIVA_PIC16, nolan-viva:VIVA_PIC16
- added J202: VIVA-HEADER-ADCNONAME, nolan-utsa:VIVA-HEADER-ADC-NONAME
- added J203: PICKIT3, nolan-viva:PICKIT3
- added J204: PINS_32.54, nolan-utsa:PINS_3
- added LED201: Hello World!, nolan-utsa:LED_RGB-5050
- added M101: VIVA_USB-TTL, nolan-utsa:VIVA_USB_TTL_SUBTEXT
- added PIC: PIC16F1829, nolan-utsa:SOP20-NEW
- added Q101: 2N3906, nolan-utsa:SOT23
- added Q102: 2N3904, nolan-utsa:SOT23
- added R101, R207: 10k, adafruit:R0805
- added R102, R206: 100k, adafruit:R0805
- added R103: 1k, adafruit:R0805
- added R104: 4k7, adafruit:R0805
- added R201, R202, R203: 150, adafruit:R0805
- added R204, R205: 2k2, adafruit:R0805
- added TP1, TP2: (no value), nolan-utsa:FIDUCIAL
- added U$201: VIVA_UTSA-KEYPAD, nolan-utsa:VIVA_UTSA-KEYPAD
- added U1: TP4056, utsa:SO08-THERMAL
- C1: value 47u -> 10u, 1206; device utsa:C-WE-5MM -> utsa:C1206
- C4: value 1u -> 47u; device utsa:C0805 -> utsa:C-WE-5MM
- C5: value 10u, 1206 -> 1u; device utsa:C1206 -> utsa:C0805
- C6: value 10u, 1206 -> 47u; device utsa:C1206 -> utsa:C-WE-5MM
- C9: value 47u -> 1u; device utsa:C-WE-5MM -> utsa:C0805
- R1: value 1k -> RPROG
- R3: value RPROG -> 1k
- U2: value AMS1117-3.3 -> AP1603; device utsa:SOT223 -> utsa:SOT23-6
- U3: value TP4056 -> AMS1117-3.3; device utsa:SO08-THERMAL -> utsa:SOT223
- moved SW1. 81.5 mm to (8.50, 68.0)
- moved L2 49.9 mm to (54.5, 86.0), turned to 180 degrees
- moved C1 47.5 mm to (22.5, 86.5), turned to 90 degrees
- moved U3 41.1 mm to (63.0, 90.0), turned to 270 degrees
- moved L1 40.6 mm to (45.5, 85.0)
- moved U2 39.7 mm to (50.0, 88.0), turned to 180 degrees
- moved F1 34.3 mm to (36.0, 86.5)
- moved LED1 31.9 mm to (26.5, 75.0), turned to 180 degrees
- moved LED2 29.7 mm to (28.5, 75.0), turned to 180 degrees
- moved C6 28.4 mm to (50.5, 80.0)
- moved C5 23.3 mm to (41.0, 88.0), turned to 270 degrees
- moved C3 22.3 mm to (47.0, 90.5), turned to 270 degrees
- moved C9 20.3 mm to (60.5, 85.0), turned to 180 degrees
- moved R1 19.7 mm to (29.0, 88.0), turned to 180 degrees
- moved C7 18.0 mm to (53.0, 91.0), turned to 270 degrees
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Connections:
- removed net DCDC_5V: C9.1+, L2.2, U5.5
- new net B+_FUSED: C4.1+, C5.2, F1.2, L1.1
- new net DCDC_OUT: C6.1+, C7.2, L2.2, U2.5
- new net DCDC_REF: C3.2, U2.3
- new net ICSP_CLK: J201.18.L, J201.18.R, J203.5, PIC.18
- new net ICSP_DAT: J201.19.L, J201.19.R, J203.4, PIC.19
- new net MCLR: J201.4.L, J201.4.R, J203.1, J204.3, PIC.4, R207.2
- new net N$10: Q102.1, R103.2
- new net N$11: LED201.4.B-, R201.1
- new net N$12: LED201.2.G-, R202.1
- new net N$13: LED201.1.R-, R203.1
- new net N$14: M101.1.3V3
- new net N$15: J102.2, Q101.3
- new net N$16: M101.6.5V
- new net N$6: J103.1, J103.2, R103.1, R104.2
- new net N$9: Q101.2, R102.1
- new net RA2: J201.17.L, J201.17.R, PIC.17, R201.2
- new net RA4: J201.3.L, J201.3.R, PIC.3, U$201.1.U
- new net RA5: J201.2.L, J201.2.R, PIC.2, R202.2
- new net RB4: J201.13.L, J201.13.R, PIC.13, R204.2
- new net RB5: J201.12.L, J201.12.R, J202.5, PIC.12
- new net RB6: J201.11.L, J201.11.R, PIC.11, R205.2
- new net RB7: J201.10.L, J201.10.R, J204.1, PIC.10
- new net RC0: J201.16.L, J201.16.R, PIC.16, U$201.4.A
- new net RC1: J201.15.L, J201.15.R, PIC.15, U$201.3.S
- new net RC2: J201.14.L, J201.14.R, J202.3, PIC.14
- new net RC3: J201.7.L, J201.7.R, J202.4, PIC.7
- new net RC4: J201.6.L, J201.6.R, M101.3.RXI, PIC.6
- new net RC5: J201.5.L, J201.5.R, M101.4.RDO, PIC.5
- new net RC6: J201.8.L, J201.8.R, PIC.8, R203.2
- new net RC7: J201.9.L, J201.9.R, PIC.9, U$201.2.T
- new net SWITCH_NODE: L1.2, U2.4
- new net VDD: C201.2, C202.2, C203.2, J201.1.L, J201.1.R, J202.2, J203.2, LED201.3.+, PIC.1, R204.1, R205.1, R206.1, R207.1
- net +3V3: now also C10.2, U3.2, U3.4.TAB; no longer C4.2, U2.2, U2.4.TAB
- net +5V: now also C8.1+, C9.2, U3.3; no longer C1.1+, C3.2, U2.3
- net B+: now also C2.+, U1.5; no longer C6.+, U3.5
- net CHARGE: now also R3.2, U1.7; no longer R2.2, U3.7
- net DCDC_ENABLE: now also U2.6; no longer U5.6
- net GND: now also B201.1.A, B201.2.A, C1.-, C10.1, C2.-, C201.1, C202.1, C203.1, C4.2-, C5.1, C6.2-, C9.1, J102.1, J201.20.L, J201.20.R, J202.1, J203.3, PIC.20, Q102.2, R1.1, R104.1, U1.1, U1.3, U1.THERMAL, U2.2; no longer C1.2-, C4.1, C5.-, C6.-, C9.2-, R3.1, U3.3, U3.THERMAL, U5.1, U5.2
- net N$1: now also B201.3.B, B201.4.B, J204.2, R206.2; no longer L1.2, U5.4
- net N$2: now also R2.1; no longer R1.1
- net N$3: now also R3.1; no longer R2.1
- net N$5: now also Q101.1, R101.2; no longer C8.1+, F1.2, L1.1
- net N$7: now also R1.2, U1.2; no longer R3.2, U3.2
- net N$8: now also Q102.3, R101.1, R102.2; no longer C7.2, U5.3
- net STANDBY: now also R2.2, U1.6; no longer R1.2, U3.6
- net USB_5V_AT: now also D1.A; no longer D3.A
- net USB_5V_PIC: now also D2.A; no longer D4.A
- net VCC: now also C1.+, D1.C, D2.C, U1.4, U1.8; no longer C5.+, D3.C, D4.C, U3.4, U3.8
Routing:
- net B+: track 0.00 -> 50.3 mm, vias 0 -> 1
- net DCDC_ENABLE: track 0.00 -> 49.2 mm, vias 0 -> 1
- net VCC: track 0.00 -> 34.4 mm, vias 0 -> 3
- net DCDC_OUT: track 0.00 -> 14.3 mm
- net +5V: track 0.00 -> 12.6 mm
- net B+_FUSED: track 0.00 -> 11.4 mm
- net +3V3: track 0.00 -> 9.83 mm
- net CHARGE: track 0.00 -> 5.69 mm
- net STANDBY: track 0.00 -> 5.52 mm
- net N$7: track 0.00 -> 2.98 mm
- net SWITCH_NODE: track 0.00 -> 2.97 mm
- net N$3: track 0.00 -> 2.58 mm
- net DCDC_REF: track 0.00 -> 2.15 mm
- net N$2: track 0.00 -> 2.08 mm

Commit message: *
Parts:
- removed C201, C202: 4u7, nolan-utsa:C0805
- removed C203: 1u, nolan-utsa:C0805
- removed J102: 1X2-3.5MM-3.5MM, nolan-utsa:1X2-3.5MM
- removed J103: PINS_2, nolan-utsa:PINS_2
- removed J201: VIVA_PIC16, nolan-viva:VIVA_PIC16
- removed J204: PINS_32.54, nolan-utsa:PINS_3
- removed M101: VIVA_USB-TTL, nolan-utsa:VIVA_USB_TTL_SUBTEXT
- removed PIC: PIC16F1829, nolan-utsa:SOP20-NEW
- removed Q101: 2N3906, nolan-utsa:SOT23
- removed Q102: 2N3904, nolan-utsa:SOT23
- removed R101, R207: 10k, adafruit:R0805
- removed R102, R206: 100k, adafruit:R0805
- removed R103: 1k, adafruit:R0805
- removed R104: 4k7, adafruit:R0805
- removed R201, R202, R203: 150, adafruit:R0805
- removed R204, R205: 2k2, adafruit:R0805
- removed TP1, TP2: (no value), nolan-utsa:FIDUCIAL
- removed U$201: VIVA_UTSA-KEYPAD, nolan-utsa:VIVA_UTSA-KEYPAD
- added C11, C12, C13, C14, C15: 1u, utsa:C0805
- added FIDUCIAL1, FIDUCIAL2: (no value), utsa:FIDUCIAL
- added J1: Transmitter, utsa:VIVA-HEADER-GPIO-RA-1
- added J2: Receiver, utsa:VIVA-HEADER-RF-RX
- added J3: Pushbutton Jumper, utsa:PINS_3
- added R10, R9: 2k2, utsa:R0805
- added R4, R5, R6: 150, utsa:R0805
- added R7, R8: 10k, utsa:R0805
- added U$11: VIVA_USB-TTL, utsa:VIVA_USB_TTL_SUBTEXT
- added U$6: VIVA_PIC16BOARD, utsa:VIVA_PIC16
- added U$7: VIVA_UTSA-KEYPADV5, utsa:VIVA_UTSA-KEYPAD-V5
- added U4: PIC16F1829, utsa:SOP20-NEW
- moved LED201 62.2 mm to (50.0, 19.0), turned to 0 degrees
Connections:
- removed net N$10: Q102.1, R103.2
- removed net N$11: LED201.4.B-, R201.1
- removed net N$12: LED201.2.G-, R202.1
- removed net N$13: LED201.1.R-, R203.1
- removed net N$15: J102.2, Q101.3
- removed net N$8: Q102.3, R101.1, R102.2
- removed net N$9: Q101.2, R102.1
- new net N$4: LED201.2.G-, R5.2
- net GND: now also C11.1, C12.1, C13.1, C14.1, C15.1, U$6.20.L, U$6.20.R, U4.20; no longer C201.1, C202.1, C203.1, J102.1, J201.20.L, J201.20.R, PIC.20, Q102.2, R104.1
- net ICSP_CLK: now also U$6.18.L, U$6.18.R, U4.18; no longer J201.18.L, J201.18.R, PIC.18
- net ICSP_DAT: now also U$6.19.L, U$6.19.R, U4.19; no longer J201.19.L, J201.19.R, PIC.19
- net MCLR: now also J3.3, R7.2, U$6.4.L, U$6.4.R, U4.4; no longer J201.4.L, J201.4.R, J204.3, PIC.4, R207.2
- net N$1: now also J3.2, R8.2; no longer J204.2, R206.2
- net N$14: now also U$11.1.3V3; no longer M101.1.3V3
- net N$16: now also U$11.6.5V; no longer M101.6.5V
- net N$5: now also LED201.1.R-, R6.2; no longer Q101.1, R101.2
- net N$6: now also LED201.4.B-, R4.2; no longer J103.1, J103.2, R103.1, R104.2
- net RA2: now also R4.1, U$6.17.L, U$6.17.R, U4.17; no longer J201.17.L, J201.17.R, PIC.17, R201.2
- net RA4: now also U$6.3.L, U$6.3.R, U$7.1, U4.3; no longer J201.3.L, J201.3.R, PIC.3, U$201.1.U
- net RA5: now also R5.1, U$6.2.L, U$6.2.R, U4.2; no longer J201.2.L, J201.2.R, PIC.2, R202.2
- net RB4: now also R10.2, U$6.13.L, U$6.13.R, U4.13; no longer J201.13.L, J201.13.R, PIC.13, R204.2
- net RB5: now also U$6.12.L, U$6.12.R, U4.12; no longer J201.12.L, J201.12.R, PIC.12
- net RB6: now also R9.2, U$6.11.L, U$6.11.R, U4.11; no longer J201.11.L, J201.11.R, PIC.11, R205.2
- net RB7: now also J3.1, U$6.10.L, U$6.10.R, U4.10; no longer J201.10.L, J201.10.R, J204.1, PIC.10
- net RC0: now also U$6.16.L, U$6.16.R, U$7.4, U4.16; no longer J201.16.L, J201.16.R, PIC.16, U$201.4.A
- net RC1: now also U$6.15.L, U$6.15.R, U$7.3, U4.15; no longer J201.15.L, J201.15.R, PIC.15, U$201.3.S
- net RC2: now also U$6.14.L, U$6.14.R, U4.14; no longer J201.14.L, J201.14.R, PIC.14
- net RC3: now also U$6.7.L, U$6.7.R, U4.7; no longer J201.7.L, J201.7.R, PIC.7
- net RC4: now also U$11.3.RXI, U$6.6.L, U$6.6.R, U4.6; no longer J201.6.L, J201.6.R, M101.3.RXI, PIC.6
- net RC5: now also U$11.4.RDO, U$6.5.L, U$6.5.R, U4.5; no longer J201.5.L, J201.5.R, M101.4.RDO, PIC.5
- net RC6: now also R6.1, U$6.8.L, U$6.8.R, U4.8; no longer J201.8.L, J201.8.R, PIC.8, R203.2
- net RC7: now also U$6.9.L, U$6.9.R, U$7.2, U4.9; no longer J201.9.L, J201.9.R, PIC.9, U$201.2.T
- net VDD: now also C11.2, C12.2, C13.2, C14.2, C15.2, R10.1, R7.1, R8.1, R9.1, U$6.1.L, U$6.1.R, U4.1; no longer C201.2, C202.2, C203.2, J201.1.L, J201.1.R, PIC.1, R204.1, R205.1, R206.1, R207.1
Routing:
- net RA5: track 0.00 -> 12.1 mm
- net RA4: track 0.00 -> 11.5 mm
- net RB7: track 0.00 -> 10.9 mm
- net RB6: track 0.00 -> 10.9 mm
- net ICSP_DAT: track 0.00 -> 10.9 mm
- net RC7: track 0.00 -> 10.4 mm
- net RB5: track 0.00 -> 10.4 mm
- net ICSP_CLK: track 0.00 -> 10.3 mm
- net RC6: track 0.00 -> 9.89 mm
- net RB4: track 0.00 -> 9.87 mm
- net MCLR: track 0.00 -> 9.83 mm
- net RA2: track 0.00 -> 9.82 mm
- net RC3: track 0.00 -> 9.36 mm
- net RC2: track 0.00 -> 9.34 mm
- net RC5: track 0.00 -> 9.31 mm
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