File: VIVA_PIC16/Rev 5.0/v5.brd (EAGLE design)
At the start: 100 x 100 mm, 31 parts, among them J1 VDD Selector, J2 Transmitter, J3 Receiver, J4 PICKIT3, J5 VIVA-HEADER-ADCNONAME, U1 VIVA_UTSA-KEYPADV5, U2 VIVA_USB-TTL, U3 PIC16F1829, U4 VIVA-HEADER-I2C-RA, U5 VIVA_PIC16BOARD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

Commit message: *
Parts:
- added C7, C8: (no value), utsa:C0805
- added J6: ICSP, utsa:PINS_6-2X3
- added J7, J8: PINS_162X8, utsa:PINS16_2X8
- added U$2: VIVA-HEADER-UART-XS, utsa:PINS_4
- added U$3: VIVA_OLED, utsa:VIVA_OLED-I2C
- added XTAL1: (no value), utsa:HC49S-SMD
- J5: value VIVA-HEADER-ADCNONAME -> (none); device nolan-utsa:VIVA-HEADER-ADC-NONAME -> utsa:VIVA-HEADER-ADC-PIC16
- LED1: value Hello World! -> (none); device nolan-utsa:LED_RGB-5050 -> utsa:0805_RGB
- moved C3 9.01 mm to (53.5, 18.5), turned to 180 degrees
- moved R3 5.10 mm to (52.0, 23.5)
- moved U4 5.00 mm to (96.0, 45.0)
- moved R1 4.12 mm to (49.0, 23.5)
- moved R2 4.12 mm to (46.0, 23.5)
- moved LED1 2.00 mm to (48.0, 19.0)
- turned U6 to 45 degrees
Connections:
- new net AT_MISO: J6.1, U6.7
- new net AT_MOSI: J6.4, U6.17
- new net AT_RESET: J6.5
- new net AT_RST: U6.29
- new net AT_SCK: J6.3, U6.8
- new net AT_VTG: J6.2
- new net N$2: C7.2, XTAL1.2, XTAL1.4
- new net N$3: C8.2, XTAL1.1, XTAL1.3
- net GND: now also C7.1, C8.1, J6.6
- net N$4: now also LED1.2, R1.2; no longer LED1.2.G-, R2.2
- net N$5: now also LED1.3, R2.2; no longer LED1.1.R-, R3.2
- net N$6: now also LED1.1, R3.2; no longer LED1.4.B-, R1.2
- net RA2: now also R3.1; no longer R1.1
- net RC6: now also R1.1; no longer R3.1
- net VDD: now also LED1.4; no longer LED1.3.+
Routing:
- net RB6: track 46.5 -> 54.1 mm
- net RB4: track 50.6 -> 58.1 mm
- net VDD: track 237.5 -> 244.7 mm
- net MCLR: track 115.2 -> 117.7 mm
- net RC2: track 44.2 -> 46.8 mm
- net ICSP_CLK: track 62.0 -> 64.6 mm
- net RC5: track 31.1 -> 33.6 mm
- net RC4: track 23.7 -> 26.2 mm
- net RB7: track 25.0 -> 27.5 mm
- net RB5: track 46.1 -> 48.6 mm
- net RA4: track 48.7 -> 51.3 mm
- net ICSP_DAT: track 61.7 -> 64.2 mm
- net N$5: track 3.72 -> 6.22 mm
- net RC6: track 17.9 -> 20.3 mm
- net N$4: track 4.10 -> 6.43 mm
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Other:
- board text added: "Hello World!"

Commit message: *
Parts:
- removed J2: Transmitter, utsa:VIVA-HEADER-GPIO-RA-1
- removed J3: Receiver, utsa:VIVA-HEADER-RF-RX
- added B3: (no value), nolan-utsa:6X6MM
- added C10: 10u, utsa:C0805
- added C11: 100n, utsa:C0805
- added C12, C13: (no value), utsa:C0805
- added C9: 1u, utsa:C0805
- added J10: ADC7, utsa:VIVA-HEADER-GPIO-RA-1
- added J11: ADC6, utsa:VIVA-HEADER-GPIO-RA-1
- added J9: (no value), utsa:VIVA-HEADER-ADC-PIC16
- added R10, R13, R9: 10k, utsa:R0805
- added R11, R12: 10, utsa:R0805
- added U7: VIVA_USB-TTL, utsa:VIVA_USB_TTL_SUBTEXT
- moved C8 84.4 mm to (43.6, 61.1), turned to 45 degrees
- moved C7 83.4 mm to (40.0, 64.5), turned to 45 degrees
- moved XTAL1 81.7 mm to (45.4, 66.6), turned to 135 degrees
- moved J6 12.6 mm to (58.5, 62.0), turned to 0 degrees
- moved U$3 4.53 mm to (15.5, 63.5)
Connections:
- net N$1 renamed MCLR_CAP
- removed net N$2: C7.2, XTAL1.2, XTAL1.4
- removed net N$3: C8.2, XTAL1.1, XTAL1.3
- removed net RB4: R5.2, U3.13, U4.3, U5.13.L, U5.13.R
- removed net RB6: R6.2, U3.11, U4.4, U5.11.L, U5.11.R
- new net ADC6: J11.3, U6.19
- new net ADC7: J10.3, U6.22
- new net AREF: C10.2, C11.2, R12.2, U6.20
- new net AT_RST_BTN: B3.3.B, B3.4.B, R13.1, R9.2
- new net AT_RST_CAP: C9.2, R10.2, R9.1
- new net AT_RXD: U6.30, U7.4.RDO
- new net AT_TXD: U6.31, U7.3.RXI
- new net AVCC: C10.1, C11.1, R11.2, U6.18
- new net PC0: J9.3, U6.23
- new net PC1: J9.4, U6.24
- new net PC2: J9.5, U6.25
- new net SCL: R6.2, U$3.3.SCL, U3.11, U4.4, U5.11.L, U5.11.R, U6.28
- new net SDA: R5.2, U$3.4.SDA, U3.13, U4.3, U5.13.L, U5.13.R, U6.27
- new net XTAL1: C7.2, U6.7, XTAL1.2, XTAL1.4
- new net XTAL2: C8.2, U6.8, XTAL1.1, XTAL1.3
- net +3V3: now also U7.1.3V3
- net +5V: now also U7.6.5V
- net AT_MISO: now also U6.16; no longer U6.7
- net AT_MOSI: now also U6.15; no longer U6.17
- net AT_RST: now also R13.2
- net AT_SCK: now also U6.17; no longer U6.8
- net GND: now also B3.1.A, B3.2.A, C12.1, C13.1, C9.1, J10.1, J11.1, J9.1, R12.1, U$3.2.GND, U7.5.GND; no longer J2.1, J3.1, U6.20
- net VDD: now also C12.2, C13.2, J10.2, J11.2, J9.2, R10.1, R11.1, U$3.1.VDD; no longer J2.2, J3.2, U6.18
Routing:
- net VDD: track 244.7 -> 379.4 mm, vias 4 -> 8
- net SDA: track 0.00 -> 58.7 mm, vias 0 -> 2
- net RB4: track 58.1 -> 0.00 mm, vias 1 -> 0
- net SCL: track 0.00 -> 54.6 mm, vias 0 -> 2
- net RB6: track 54.1 -> 0.00 mm, vias 1 -> 0
- net ADC6: track 0.00 -> 37.8 mm, vias 0 -> 2
- net AT_MOSI: track 0.00 -> 35.3 mm
- net ADC7: track 0.00 -> 29.5 mm, vias 0 -> 2
- net +3V3: track 10.7 -> 40.2 mm
- net AT_RST_BTN: track 0.00 -> 28.8 mm
- net AT_SCK: track 0.00 -> 24.6 mm, vias 0 -> 2
- net +5V: track 28.0 -> 51.0 mm, vias 1 -> 2
- net AT_RXD: track 0.00 -> 22.1 mm
- net PC0: track 0.00 -> 21.0 mm, vias 0 -> 2
- net AT_TXD: track 0.00 -> 20.6 mm
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Other:
- board text added: "RESET"
- board text removed: "MCLR"
