File: VIVA_PIC16/Rev 5.0/v5-pi.brd (EAGLE design)
At the start: 100 x 100 mm, 63 parts, among them J1 VDD Selector, J2 A, J4 PICKIT3, J6 ICSP, U1 VIVA_UTSA-KEYPADV5, U2 VIVA_USB-TTL, U3 PIC16F1829, U4 VIVA-HEADER-I2C-RA, U5 VIVA_PIC16BOARD, U6 ATMEGA328-AU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

Commit message: *
Parts:
- added J8-: RPI ZERO, utsa:RPI_ZERO
- J3: value (none) -> B
- moved U4 56.4 mm to (51.0, 53.5), turned to 0 degrees
- moved C6 3.54 mm to (52.5, 57.0)
- moved R5 3.54 mm to (54.5, 59.5)
- moved R6 3.54 mm to (54.5, 62.0)
- moved C16 0.50 mm to (20.0, 88.0)
Connections:
- net +5V: now also J8-.2, J8-.4
- net GND: now also J8-.14, J8-.20, J8-.25, J8-.30, J8-.34, J8-.39, J8-.6, J8-.9
- net SCL: now also J8-.5
- net SDA: now also J8-.3
Routing:
- net +5V: track 94.9 -> 193.8 mm, vias 3 -> 5
- net VDD: track 473.5 -> 445.0 mm, vias 28 -> 27
- net SDA: track 213.9 -> 207.3 mm, vias 10 -> 8
- net SCL: track 218.9 -> 213.4 mm, vias 9 -> 7
- net ADC7: track 29.1 -> 28.5 mm
Other:
- board text added: "1"
- board text added: "RPI ZERO"
