File: VIVA_PIC16/Rev 5.0/v5-pi.sch (EAGLE design)
At the start: 63 parts, among them J1 VDD Selector, J2 A, J3 PINS_4_0100, J4 PICKIT3, J6 ICSP, U1 VIVA_UTSA-KEYPADV5, U2 VIVA_USB-TTL, U3 PIC16F1829, U4 VIVA-HEADER-I2C-RA, U5 VIVA_PIC16BOARD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

Commit message: *
Parts:
- added J8-: RPI ZERO, utsa:RPI_ZERO
- J3: value PINS_4_0100 -> B
Connections:
- net +5V: now also J8-2_(5V).1, J8-4_(5V).1
- net GND: now also J8-14_(GND).1, J8-20_(GND).1, J8-25_(GND).1, J8-30_(GND).1, J8-34_(GND).1, J8-39_(GND).1, J8-6_(GND).1, J8-9_(GND).1
- net SCL: now also J8-5_(GPIO3).1
- net SDA: now also J8-3_(GPIO2).1
Other:
- note added: "433MHz RECEIVER: MX-05V"
- note added: "433MHz TRANSMITTER: MX-FS-03V"
- note added: "FOR ID EEPROM ONLY"
