File: VIVA_PIC16/Rev DRAFT/VIVA PIC16 with battery.brd (EAGLE design)
At the start: 100 x 100 mm, 31 parts, among them J1 VDD Selector, J2 Transmitter, J3 Receiver, J4 PICKIT3, J5 VIVA-HEADER-ADCNONAME, U1 VIVA_UTSA-KEYPADV5, U2 VIVA_USB-TTL, U3 PIC16F1829, U4 VIVA-HEADER-I2C-RA, U5 VIVA_PIC16BOARD, U6 ATMEGA328-AU

Commit message: *
Parts:
- removed B2: (no value), nolan-utsa:6X6MM
- removed J4: PICKIT3, nolan-viva:PICKIT3
- removed J5: VIVA-HEADER-ADCNONAME, nolan-utsa:VIVA-HEADER-ADC-NONAME
- removed U6: ATMEGA328-AU, utsa:32A_ATM
- added B201: (no value), nolan-utsa:6X6MM
- added C10, C11, C12, C13, C14, C15, C7, C9: 1u, utsa:C0805
- added C8: 47u, utsa:C-WE-5MM
- added D1, D2: 1N5819, utsa:SOD80C
- added F1: 0805, utsa:F0805
- added J202: VIVA-HEADER-ADCNONAME, nolan-utsa:VIVA-HEADER-ADC-NONAME
- added J203: PICKIT3, nolan-viva:PICKIT3
- added L1, L2: 22u, utsa:SRN5040
- added LED2: CHG, utsa:CHIPLED_0603
- added LED201: Hello World!, nolan-utsa:LED_RGB-5050
- added R10, R9: 2k2, utsa:R0805
- added SW1.: OS202013MT5QN1, utsa:OS202013MT5QN1
- added U$11: VIVA_USB-TTL, utsa:VIVA_USB_TTL_SUBTEXT
- added U$7: VIVA_UTSA-KEYPADV5, utsa:VIVA_UTSA-KEYPAD-V5
- B1: value (none) -> 1043; device nolan-utsa:6X6MM -> utsa:BATTERY-18650-1
- C1, C2: value 1u -> 10u, 1206; device utsa:C0805 -> utsa:C1206
- C4, C6: value 1u -> 47u; device utsa:C0805 -> utsa:C-WE-5MM
- J1: value VDD Selector -> Transmitter; device utsa:PINS_3 -> utsa:VIVA-HEADER-GPIO-RA-1
- J2: value Transmitter -> Receiver; device utsa:VIVA-HEADER-GPIO-RA-1 -> utsa:VIVA-HEADER-RF-RX
- J3: value Receiver -> Pushbutton Jumper; device utsa:VIVA-HEADER-RF-RX -> utsa:PINS_3
- LED1: value Hello World! -> SBY; device nolan-utsa:LED_RGB-5050 -> utsa:CHIPLED_0603
- R1: value 150 -> RPROG
- R2, R3: value 150 -> 1k
- R4: value 10k -> 150
- R5, R6: value 2k2 -> 150
- U1: value VIVA_UTSA-KEYPADV5 -> TP4056; device utsa:VIVA_UTSA-KEYPAD-V5 -> utsa:SO08-THERMAL
- U2: value VIVA_USB-TTL -> AP1603; device utsa:VIVA_USB_TTL_SUBTEXT -> utsa:SOT23-6
- U3: value PIC16F1829 -> AMS1117-3.3; device utsa:SOP20-NEW -> utsa:SOT223
- U4: value VIVA-HEADER-I2C-RA -> PIC16F1829; device utsa:VIVA-HEADER-I2C-RA -> utsa:SOP20-NEW
- moved J2 88.6 mm to (94.0, 60.0), turned to 270 degrees
- moved J1 88.1 mm to (94.0, 74.0), turned to 270 degrees
- moved U1 84.1 mm to (27.5, 82.5), turned to 180 degrees
- moved B1 78.0 mm to (50.0, 85.0), flipped to the bottom, turned to 180 degrees
- moved C5 75.9 mm to (41.0, 88.0), turned to 270 degrees
- moved C3 71.5 mm to (47.0, 90.5), turned to 270 degrees
- moved R1 69.8 mm to (29.0, 88.0), turned to 180 degrees
- moved C6 65.6 mm to (50.5, 80.0), turned to 0 degrees
- moved LED1 60.7 mm to (26.5, 75.0), turned to 180 degrees
- moved J3 60.3 mm to (18.0, 15.0)
- moved C4 59.2 mm to (39.5, 81.5)
- moved U2 58.8 mm to (50.0, 88.0), turned to 180 degrees
- moved U3 58.5 mm to (63.0, 90.0)
- moved R2 58.4 mm to (24.5, 75.0), turned to 90 degrees
- moved R3 54.9 mm to (31.0, 75.0), turned to 90 degrees
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- renumbered U5 to U$6
Connections:
- new net B+: B1.+, C2.+, F1.1, SW1..1, U1.5
- new net B+_FUSED: C4.1+, C5.2, F1.2, L1.1
- new net CHARGE: R3.2, U1.7
- new net DCDC_ENABLE: SW1..2, U2.6
- new net DCDC_OUT: C6.1+, C7.2, L2.2, U2.5
- new net DCDC_REF: C3.2, U2.3
- new net N$14: U$11.1.3V3
- new net N$16: U$11.6.5V
- new net N$2: LED1.C, R2.1
- new net N$3: LED2.C, R3.1
- new net N$7: R1.2, U1.2
- new net STANDBY: R2.2, U1.6
- new net SWITCH_NODE: L1.2, U2.4
- new net USB_5V_AT: D1.A
- new net USB_5V_PIC: D2.A
- new net VCC: C1.+, D1.C, D2.C, LED1.A, LED2.A, U1.4, U1.8
- net +3V3: now also C10.2, U3.2, U3.4.TAB; no longer J1.1, U2.1.3V3
- net +5V: now also C8.1+, C9.2, L2.1, U3.3; no longer J1.3, U2.6.5V
- net GND: now also B1.1, B201.1.A, B201.2.A, C1.-, C10.1, C11.1, C12.1, C13.1, C14.1, C15.1, C2.-, C4.2-, C6.2-, C7.1, C8.2-, C9.1, J202.1, J203.3, R1.1, SW1..3, U1.1, U1.3, U1.THERMAL, U2.1, U2.2, U3.1, U4.20; no longer B1.1.A, B1.2.A, B2.1.A, B2.2.A, C1.1, C2.1, C4.1, C6.1, J2.1, J3.1, J4.3, J5.1, U2.5.GND, U3.20, U4.1, U6.20, U6.21, U6.3, U6.5
- net ICSP_CLK: now also J203.5, U4.18; no longer J4.5, U3.18
- net ICSP_DAT: now also J203.4, U4.19; no longer J4.4, U3.19
- net MCLR: now also J203.1, J3.3, U4.4; no longer B2.3.B, B2.4.B, J4.1, U3.4
- net N$1: now also B201.3.B, B201.4.B, J3.2; no longer C5.2, R7.1
- net N$4: now also LED201.2.G-, R5.2; no longer LED1.2.G-, R2.2
- net N$5: now also LED201.1.R-, R6.2; no longer LED1.1.R-, R3.2
- net N$6: now also LED201.4.B-, R4.2; no longer LED1.4.B-, R1.2
- net RA2: now also R4.1, U4.17; no longer R1.1, U3.17
- net RA4: now also U$7.1, U4.3; no longer U1.1, U3.3
- net RA5: now also R5.1, U4.2; no longer R2.1, U3.2
- net RB4: now also R10.2, U4.13; no longer R5.2, U3.13, U4.3
- net RB5: now also J202.5, U4.12; no longer J5.5, U3.12
- net RB6: now also R9.2, U4.11; no longer R6.2, U3.11, U4.4
- net RB7: now also J3.1, U4.10; no longer B1.3.B, B1.4.B, C4.2, R4.2, U3.10
- net RC0: now also U$7.4, U4.16; no longer U1.4, U3.16
- net RC1: now also U$7.3, U4.15; no longer U1.3, U3.15
- net RC2: now also J202.3, U4.14; no longer J5.3, U3.14
- net RC3: now also J202.4, U4.7; no longer J5.4, U3.7
- net RC4: now also U$11.3.RXI, U4.6; no longer U2.3.RXI, U3.6
- net RC5: now also U$11.4.RDO, U4.5; no longer U2.4.RDO, U3.5
- net RC6: now also R6.1, U4.8; no longer R3.1, U3.8
- net RC7: now also U$7.2, U4.9; no longer U1.2, U3.9
- net VDD: now also C11.2, C12.2, C13.2, C14.2, C15.2, J202.2, J203.2, LED201.3.+, R10.1, R7.1, R9.1, U4.1; no longer C1.2, C2.2, C3.2, C6.2, J1.2, J2.2, J3.2, J4.2, J5.2, LED1.3.+, R4.1, R5.1, R6.1, U3.1, U4.2, U6.18, U6.4, U6.6
Routing:
- net VDD: track 237.5 -> 3.59 mm, vias 4 -> 0
- net MCLR: track 115.2 -> 9.83 mm, vias 2 -> 0
- net RC3: track 71.5 -> 9.36 mm, vias 4 -> 0
- net ICSP_CLK: track 62.0 -> 10.3 mm, vias 2 -> 0
- net ICSP_DAT: track 61.7 -> 10.9 mm, vias 1 -> 0
- net B+: track 0.00 -> 50.3 mm, vias 0 -> 1
- net DCDC_ENABLE: track 0.00 -> 49.2 mm, vias 0 -> 1
- net RB4: track 50.6 -> 9.87 mm, vias 1 -> 0
- net RA4: track 48.7 -> 11.5 mm
- net RB5: track 46.1 -> 10.4 mm, vias 1 -> 0
- net RB6: track 46.5 -> 10.9 mm, vias 1 -> 0
- net RC2: track 44.2 -> 9.34 mm
- net VCC: track 0.00 -> 34.4 mm, vias 0 -> 3
- net RC1: track 41.4 -> 8.88 mm, vias 1 -> 0
- net RC0: track 40.5 -> 9.29 mm
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Other:
- board text removed: "3V3"
- board text removed: "5V"
- board text removed: "MCLR"
- board text removed: "RB7"
