File: VIVA_PIC16/Rev DRAFT/VIVA PIC16 with battery.sch (EAGLE design)
At the start: 31 parts, among them J1 VDD Selector, J2 Transmitter, J3 Receiver, J4 PICKIT3, J5 VIVA-HEADER-ADCNONAME, U1 VIVA_UTSA-KEYPADV5, U2 VIVA_USB-TTL, U3 PIC16F1829, U4 VIVA-HEADER-I2C-RA, U5 VIVA_PIC16BOARD, U6 ATMEGA328-AU

Commit message: *
Parts:
- removed B2: (no value), nolan-utsa:PUSHBUTTON6X6MM
- removed J4: PICKIT3, nolan-viva:PICKIT3
- removed J5: VIVA-HEADER-ADCNONAME, nolan-utsa:VIVA-HEADER-ADCNONAME
- removed U5: VIVA_PIC16BOARD, utsa:VIVA_PIC16BOARD
- removed U6: ATMEGA328-AU, utsa:ATMEGA328-AU
- added B201: (no value), nolan-utsa:PUSHBUTTON6X6MM
- added C10, C11, C12, C13, C14, C15, C7, C9: 1u, utsa:C0805
- added C8: 47u, utsa:C-EU865080642006
- added D1, D2: 1N5819, utsa:DIODE-SOD80C
- added F1: 0805, utsa:FUSE0805
- added J202: VIVA-HEADER-ADCNONAME, nolan-utsa:VIVA-HEADER-ADCNONAME
- added J203: PICKIT3, nolan-viva:PICKIT3
- added L1, L2: 22u, utsa:L5040
- added LED2: CHG, utsa:LEDCHIPLED_0603
- added LED201: Hello World!, nolan-utsa:RGB_LED
- added R10, R9: 2k2, utsa:R-EU__R0805
- added SW1.: OS202013MT5QN1, utsa:SWITCH_DPDT
- added U$11: VIVA_USB-TTL, utsa:VIVA_USB-TTL
- added U$6: VIVA_PIC16BOARD, utsa:VIVA_PIC16BOARD
- added U$7: VIVA_UTSA-KEYPADV5, utsa:VIVA_UTSA-KEYPADV5
- B1: value (none) -> 1043; device nolan-utsa:PUSHBUTTON6X6MM -> utsa:BATTERY18650
- C1, C2: value 1u -> 10u, 1206; device utsa:C0805 -> utsa:C-EUC1206
- C4, C6: value 1u -> 47u; device utsa:C0805 -> utsa:C-EU865080642006
- J1: value VDD Selector -> Transmitter; device utsa:PINS_3_2.54 -> utsa:VIVA-HEADER-GPIO-1
- J2: value Transmitter -> Receiver; device utsa:VIVA-HEADER-GPIO-1 -> utsa:VIVA-HEADER-RF-RX
- J3: value Receiver -> Pushbutton Jumper; device utsa:VIVA-HEADER-RF-RX -> utsa:PINS_3_2.54
- LED1: value Hello World! -> SBY; device nolan-utsa:RGB_LED -> utsa:LEDCHIPLED_0603
- R1: value 150 -> RPROG
- R2, R3: value 150 -> 1k
- R4: value 10k -> 150
- R5, R6: value 2k2 -> 150
- U1: value VIVA_UTSA-KEYPADV5 -> TP4056; device utsa:VIVA_UTSA-KEYPADV5 -> utsa:TP4056
- U2: value VIVA_USB-TTL -> AP1603; device utsa:VIVA_USB-TTL -> utsa:AP1603
- U3: value PIC16F1829 -> AMS1117-3.3; device utsa:PIC16F1829300 -> utsa:REGULATOR_SCHLM1117
- U4: value VIVA-HEADER-I2C-RA -> PIC16F1829; device utsa:VIVA-HEADER-I2C-RA -> utsa:PIC16F1829300
Connections:
- new net B+: B1.+, C2.1, F1.1, SW1.A.ON, U1.5.BAT
- new net B+_FUSED: C4.1, C5.+, F1.2, L1.1
- new net CHARGE: R3.2, U1.7.CHRG
- new net DCDC_ENABLE: SW1.A.IN, U2.6.EN
- new net DCDC_OUT: C6.1, C7.+, L2.2, U2.5.OUT
- new net DCDC_REF: C3.+, U2.3.REF
- new net N$14: U$11.(1)3V3
- new net N$16: U$11.(6)5V
- new net N$2: LED1.C, R2.1
- new net N$3: LED2.C, R3.1
- new net N$7: R1.2, U1.2.PROG
- new net STANDBY: R2.2, U1.6.STDBY
- new net SWITCH_NODE: L1.2, U2.4.LX
- new net USB_5V_AT: D1.A
- new net USB_5V_PIC: D2.A
- new net VCC: C1.1, D1.C, D2.C, LED1.A, LED2.A, U1.4.VCC, U1.8.ENABLE
- net +3V3: now also C10.+, U3.OUT; no longer J1.1, U2.(1)3V3
- net +5V: now also C8.1, C9.+, L2.1, U3.IN; no longer J1.3, U2.(6)5V
- net GND: now also B1.-, B201.1, C1.2, C10.-, C11.-, C12.-, C13.-, C14.-, C15.-, C2.2, C4.2, C6.2, C7.-, C8.2, C9.-, J202.1.GND, J203.3.VSS(GND), R1.1, SW1.A.OFF, U$6.20, U1.1.TEMP, U1.3.GND, U2.1.FB, U2.2.GND, U3.GND, U4.20.VSS; no longer B1.1, B2.1, C1.-, C2.-, C4.-, C6.-, J2.1.GND, J3.1.GND, J4.3.VSS(GND), J5.1.GND, U2.(5)GND, U3.20.VSS, U4.1.GND, U5.20, U6.AREF, U6.GND, U6.GND_2, U6.GND_3
- net ICSP_CLK: now also J203.5.PGC, U$6.18, U4.18.RA1/ICSPCLK; no longer J4.5.PGC, U3.18.RA1/ICSPCLK, U5.18
- net ICSP_DAT: now also J203.4.PGD, U$6.19, U4.19.RA0/ICSPDAT; no longer J4.4.PGD, U3.19.RA0/ICSPDAT, U5.19
- net MCLR: now also J203.1.MCLR, J3.3, U$6.4, U4.4.RA3/MCLR; no longer B2.2, J4.1.MCLR, U3.4.RA3/MCLR, U5.4
- net N$1: now also B201.2, J3.2; no longer C5.+, R7.1
- net N$4: now also LED201.2.G-, R5.2; no longer LED1.2.G-, R2.2
- net N$5: now also LED201.1.R-, R6.2; no longer LED1.1.R-, R3.2
- net N$6: now also LED201.4.B-, R4.2; no longer LED1.4.B-, R1.2
- net RA2: now also R4.1, U$6.17, U4.17.RA2; no longer R1.1, U3.17.RA2, U5.17
- net RA4: now also U$6.3, U$7.1, U4.3.RA4; no longer U1.1, U3.3.RA4, U5.3
- net RA5: now also R5.1, U$6.2, U4.2.RA5; no longer R2.1, U3.2.RA5, U5.2
- net RB4: now also R10.2, U$6.13, U4.13.RB4; no longer R5.2, U3.13.RB4, U4.3.SDA, U5.13
- net RB5: now also J202.5.ADC2, U$6.12, U4.12.RB5; no longer J5.5.ADC2, U3.12.RB5, U5.12
- net RB6: now also R9.2, U$6.11, U4.11.RB6; no longer R6.2, U3.11.RB6, U4.4.SCL, U5.11
- net RB7: now also J3.1, U$6.10, U4.10.RB7; no longer B1.2, C4.+, R4.2, U3.10.RB7, U5.10
- net RC0: now also U$6.16, U$7.4, U4.16.RC0; no longer U1.4, U3.16.RC0, U5.16
- net RC1: now also U$6.15, U$7.3, U4.15.RC1; no longer U1.3, U3.15.RC1, U5.15
- net RC2: now also J202.3.ADC0, U$6.14, U4.14.RC2; no longer J5.3.ADC0, U3.14.RC2, U5.14
- net RC3: now also J202.4.ADC1, U$6.7, U4.7.RC3; no longer J5.4.ADC1, U3.7.RC3, U5.7
- net RC4: now also U$11.(3)MCU.TX, U$6.6, U4.6.RC4; no longer U2.(3)MCU.TX, U3.6.RC4, U5.6
- net RC5: now also U$11.(4)MCU.RX, U$6.5, U4.5.RC5; no longer U2.(4)MCU.RX, U3.5.RC5, U5.5
- net RC6: now also R6.1, U$6.8, U4.8.RC6; no longer R3.1, U3.8.RC6, U5.8
- net RC7: now also U$6.9, U$7.2, U4.9.RC7; no longer U1.2, U3.9.RC7, U5.9
- net VDD: now also C11.+, C12.+, C13.+, C14.+, C15.+, J202.2.VDD, J203.2.VDD(PWR), LED201.3.+, R10.1, R7.1, R9.1, U$6.1, U4.1.VDD; no longer C1.+, C2.+, C3.+, C6.+, J1.2, J2.2.VDD, J3.2.VDD, J4.2.VDD(PWR), J5.2.VDD, LED1.3.+, R4.1, R5.1, R6.1, U3.1.VDD, U4.2.VDD, U5.1, U6.AVCC, U6.VCC, U6.VCC_2
Other:
- note added: "Fiducials"
- note added: "Keystone Electronics 1 cell, 18650"
- note added: "NOTES: (1) Shielded end of switching power supply inductor is connected to switch node."
- note added: "Push Button"
- note added: "VIVA Header: ANALOG"
- note added: "switch node"
- note removed: "Fiducial"
- note removed: "General Purpose Button"
- note removed: "Reset Button"
